File: full.sch (EAGLE design)
At the start: 20 parts, among them J1 Audio PC, J2 Audio Radio, T1 2N3440, X1 PTT

Commit message: Supply LED | Supply Switch
Parts:
- added LED1: LAP4-TOP, led:LAP4-TOP
- added R10: (no value), rcl:R-US_0204/2V
- added S1: (no value), switch:255SB
Connections:
- new net N$13: LED1.A, R10.1
- new net USB_SUPPLY: S1.P
- net +5V: now also R10.2, S1.S
- net 0: now also LED1.C
Other:
- moved on the sheet: C2, J2
Changed lines of the file:
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@@
 <schematic_group name="PC_TO_RADIO"/>
 <schematic_group name="PTT"/>
+<schematic_group name="SUPPLY_TOGGLE"/>
+<schematic_group name="POWER_LAMP"/>
 </groups>
 <parts>
@@
 <part name="X_7" library="ngspice-simulation" library_urn="urn:adsk.eagle:library:527439" deviceset="GND" device=""/>
 <part name="R9" library="rcl" library_urn="urn:adsk.eagle:library:334" deviceset="R-US_" device="0204/2V" package3d_urn="urn:adsk.eagle:package:23495/1" value="1Meg"/>
+<part name="S1" library="switch" library_urn="urn:adsk.eagle:library:380" deviceset="255SB" device="" package3d_urn="urn:adsk.eagle:package:27679/1"/>
+<part name="P+5" library="supply1" library_urn="urn:adsk.eagle:library:371" deviceset="+5V" device=""/>
+<part name="P+6" library="supply1" library_urn="urn:adsk.eagle:library:371" deviceset="+5V" device=""/>
+<part name="X_8" library="ngspice-simulation" library_urn="urn:adsk.eagle:library:527439" deviceset="GND" device=""/>
+<part name="LED1" library="led" library_urn="urn:adsk.eagle:library:259" deviceset="*P4" device="-TOP" package3d_urn="urn:adsk.eagle:package:15879/1" technology="LA" value=""/>
+<part name="R10" library="rcl" library_urn="urn:adsk.eagle:library:334" deviceset="R-US_" device="0204/2V" package3d_urn="urn:adsk.eagle:package:23495/1"/>
 </parts>
 <sheets>
@@
 <attribute name="VALUE" x="-81.28" y="62.23" size="1.778" layer="96"/>
 </instance>
-<instance part="J2" gate="G$1" x="-73.66" y="-17.78" smashed="yes" grouprefs="RADIO_TO_PC">
-<attribute name="NAME" x="-76.2" y="-13.97" size="1.778" layer="95"/>
-<attribute name="VALUE" x="-76.2" y="-24.13" size="1.778" layer="96"/>
+<instance part="J2" gate="G$1" x="-76.2" y="27.94" smashed="yes" grouprefs="RADIO_TO_PC">
+<attribute name="NAME" x="-78.74" y="31.75" size="1.778" layer="95"/>
+<attribute name="VALUE" x="-78.74" y="21.59" size="1.778" layer="96"/>
 </instance>
 <instance part="X_1" gate="G$1" x="-66.04" y="58.42" smashed="yes" grouprefs="PC_TO_RADIO"/>
-<instance part="X_2" gate="G$1" x="-60.96" y="-25.4" smashed="yes" grouprefs="RADIO_TO_PC"/>
+<instance part="X_2" gate="G$1" x="-63.5" y="20.32" smashed="yes" grouprefs="RADIO_TO_PC"/>
 <instance part="X_3" gate="G$1" x="48.26" y="43.18" smashed="yes"/>
 <instance part="C1" gate="G$1" x="-40.64" y="53.34" smashed="yes" rot="R180" grouprefs="PC_TO_RADIO">
@@
 <attribute name="VALUE" x="-42.164" y="58.039" size="1.778" layer="96" rot="R180"/>
 </instance>
-<instance part="C2" gate="G$1" x="-50.8" y="-17.78" smashed="yes" rot="R90" grouprefs="RADIO_TO_PC">
-<attribute name="NAME" x="-51.181" y="-16.256" size="1.778" layer="95" rot="R90"/>
-<attribute name="VALUE" x="-46.101" y="-16.256" size="1.778" layer="96" rot="R90"/>
+<instance part="C2" gate="G$1" x="-53.34" y="27.94" smashed="yes" rot="R90" grouprefs="RADIO_TO_PC">
+<attribute name="NAME" x="-53.721" y="29.464" size="1.778" layer="95" rot="R90"/>
+<attribute name="VALUE" x="-48.641" y="29.464" size="1.778" layer="96" rot="R90"/>
 </instance>
 <instance part="P+1" gate="1" x="48.26" y="55.88" smashed="yes">
@@
 <attribute name="NAME" x="150.9014" y="41.91" size="1.778" layer="95" rot="R90"/>
 <attribute name="VALUE" x="155.702" y="41.91" size="1.778" layer="96" rot="R90"/>
+</instance>
+<instance part="S1" gate="1" x="78.74" y="111.76" smashed="yes" rot="R270" grouprefs="SUPPLY_TOGGLE">
+<attribute name="NAME" x="76.835" y="118.11" size="1.778" layer="95"/>
+<attribute name="VALUE" x="81.915" y="115.57" size="1.778" layer="96"/>
+</instance>
+<instance part="P+5" gate="1" x="88.9" y="109.22" smashed="yes" grouprefs="SUPPLY_TOGGLE">
+<attribute name="VALUE" x="86.36" y="104.14" size="1.778" layer="96" rot="R90"/>
+</instance>
+<instance part="P+6" gate="1" x="106.68" y="119.38" smashed="yes" grouprefs="POWER_LAMP">
+<attribute name="VALUE" x="104.14" y="114.3" size="1.778" layer="96" rot="R90"/>
+</instance>
+<instance part="X_8" gate="G$1" x="106.68" y="96.52" smashed="yes" grouprefs="POWER_LAMP"/>
+<instance part="LED1" gate="G$1" x="106.68" y="101.6" smashed="yes" grouprefs="POWER_LAMP">
+<attribute name="NAME" x="110.236" y="97.028" size="1.778" layer="95" rot="R90"/>
+<attribute name="VALUE" x="112.395" y="97.028" size="1.778" layer="96" rot="R90"/>
+</instance>
+<instance part="R10" gate="G$1" x="106.68" y="111.76" smashed="yes" rot="R90" grouprefs="POWER_LAMP">
+<attribute name="NAME" x="105.1814" y="107.95" size="1.778" layer="95" rot="R90"/>
+<attribute name="VALUE" x="109.982" y="107.95" size="1.778" layer="96" rot="R90"/>
 </instance>
 </instances>
@@
 <pinref part="J2" gate="G$1" pin="3"/>
 <pinref part="X_2" gate="G$1" pin="0"/>
-<wire x1="-66.04" y1="-20.32" x2="-60.96" y2="-20.32" width="0.1524" layer="91" grouprefs="RADIO_TO_PC"/>
-<wire x1="-60.96" y1="-20.32" x2="-60.96" y2="-25.4" width="0.1524" layer="91" grouprefs="RADIO_TO_PC"/>
+<wire x1="-68.58" y1="25.4" x2="-63.5" y2="25.4" width="0.1524" layer="91" grouprefs="RADIO_TO_PC"/>
+<wire x1="-63.5" y1="25.4" x2="-63.5" y2="20.32" width="0.1524" layer="91" grouprefs="RADIO_TO_PC"/>
 </segment>
 <segment>
@@
 <wire x1="165.1" y1="40.64" x2="152.4" y2="40.64" width="0.1524" layer="91" grouprefs="PTT"/>
 </segment>
+<segment>
+<pinref part="X_8" gate="G$1" pin="0"/>
+<pinref part="LED1" gate="G$1" pin="C"/>
+</segment>
 </net>
 <net name="N$1" class="0">
@@
 <segment>
 <pinref part="J2" gate="G$1" pin="2"/>
-<wire x1="-66.04" y1="-17.78" x2="-60.96" y2="-17.78" width="0.1524" layer="91" grouprefs="RADIO_TO_PC"/>
+<wire x1="-68.58" y1="27.94" x2="-63.5" y2="27.94" width="0.1524" layer="91" grouprefs="RADIO_TO_PC"/>
 <pinref part="J2" gate="G$1" pin="1"/>
-<wire x1="-60.96" y1="-15.24" x2="-66.04" y2="-15.24" width="0.1524" layer="91" grouprefs="RADIO_TO_PC"/>
-<wire x1="-60.96" y1="-17.78" x2="-60.96" y2="-15.24" width="0.1524" layer="91" grouprefs="RADIO_TO_PC"/>
+<wire x1="-63.5" y1="30.48" x2="-68.58" y2="30.48" width="0.1524" layer="91" grouprefs="RADIO_TO_PC"/>
+<wire x1="-63.5" y1="27.94" x2="-63.5" y2="30.48" width="0.1524" layer="91" grouprefs="RADIO_TO_PC"/>
 <pinref part="C2" gate="G$1" pin="1"/>
-<wire x1="-60.96" y1="-17.78" x2="-53.34" y2="-17.78" width="0.1524" layer="91" grouprefs="RADIO_TO_PC"/>
-<junction x="-60.96" y="-17.78" grouprefs="RADIO_TO_PC"/>
+<wire x1="-63.5" y1="27.94" x2="-55.88" y2="27.94" width="0.1524" layer="91" grouprefs="RADIO_TO_PC"/>
+<junction x="-63.5" y="27.94" grouprefs="RADIO_TO_PC"/>
 </segment>
 </net>
@@
 <segment>
 <pinref part="C2" gate="G$1" pin="2"/>
-<wire x1="-45.72" y1="-17.78" x2="-35.56" y2="-17.78" width="0.1524" layer="91" grouprefs="RADIO_TO_PC"/>
-<label x="-35.56" y="-17.78" size="1.778" layer="95" grouprefs="RADIO_TO_PC"/>
+<wire x1="-48.26" y1="27.94" x2="-38.1" y2="27.94" width="0.1524" layer="91" grouprefs="RADIO_TO_PC"/>
+<label x="-38.1" y="27.94" size="1.778" layer="95" grouprefs="RADIO_TO_PC"/>
 </segment>
 </net>
@@
 <wire x1="40.64" y1="15.24" x2="22.86" y2="15.24" width="0.1524" layer="91"/>
 <junction x="22.86" y="15.24"/>
+</segment>
+<segment>
+<pinref part="S1" gate="1" pin="S"/>
+<pinref part="P+5" gate="1" pin="+5V"/>
+<wire x1="83.82" y1="106.68" x2="88.9" y2="106.68" width="0.1524" layer="91" grouprefs="SUPPLY_TOGGLE"/>
+</segment>
+<segment>
+<pinref part="P+6" gate="1" pin="+5V"/>
+<pinref part="R10" gate="G$1" pin="2"/>
 </segment>
 </net>
@@
 </segment>
 </net>
+<net name="USB_SUPPLY" class="0">
+<segment>
+<pinref part="S1" gate="1" pin="P"/>
+<wire x1="73.66" y1="109.22" x2="58.42" y2="109.22" width="0.1524" layer="91" grouprefs="SUPPLY_TOGGLE"/>
+<wire x1="58.42" y1="109.22" x2="58.42" y2="114.3" width="0.1524" layer="91" grouprefs="SUPPLY_TOGGLE"/>
+<label x="58.42" y="114.3" size="1.778" layer="95" grouprefs="SUPPLY_TOGGLE"/>
+</segment>
+</net>
+<net name="N$13" class="0">
+<segment>
+<pinref part="LED1" gate="G$1" pin="A"/>
+<pinref part="R10" gate="G$1" pin="1"/>
+<wire x1="106.68" y1="104.14" x2="106.68" y2="106.68" width="0.1524" layer="91" grouprefs="POWER_LAMP"/>
+</segment>
+</net>

Commit message: Values for VOX and Optocoupler
Parts:
- C1, C2, C3: value (none) -> 100u
- OK1: value SFH618A-2 -> LTV817
- R1: value (none) -> 904
- R10: value (none) -> 150
- R2: value (none) -> 285
- R3: value (none) -> 25
- R4: value (none) -> 125
- R8: value (none) -> 220
- T1: value 2N3440 -> SC 945
Connections:
- net 0: now also U$1.GND2
Other:
- note added: "Ic = 20mA"
Changed lines of the file:
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@@
 <part name="X_2" library="ngspice-simulation" library_urn="urn:adsk.eagle:library:527439" deviceset="GND" device=""/>
 <part name="X_3" library="ngspice-simulation" library_urn="urn:adsk.eagle:library:527439" deviceset="GND" device=""/>
-<part name="C1" library="rcl" library_urn="urn:adsk.eagle:library:334" deviceset="C-EU" device="025-024X044" package3d_urn="urn:adsk.eagle:package:23630/1"/>
-<part name="C2" library="rcl" library_urn="urn:adsk.eagle:library:334" deviceset="C-EU" device="025-024X044" package3d_urn="urn:adsk.eagle:package:23630/1"/>
+<part name="C1" library="rcl" library_urn="urn:adsk.eagle:library:334" deviceset="C-EU" device="025-024X044" package3d_urn="urn:adsk.eagle:package:23630/1" value="100u"/>
+<part name="C2" library="rcl" library_urn="urn:adsk.eagle:library:334" deviceset="C-EU" device="025-024X044" package3d_urn="urn:adsk.eagle:package:23630/1" value="100u"/>
 <part name="P+1" library="supply1" library_urn="urn:adsk.eagle:library:371" deviceset="+5V" device=""/>
-<part name="C3" library="rcl" library_urn="urn:adsk.eagle:library:334" deviceset="C-EU" device="025-024X044" package3d_urn="urn:adsk.eagle:package:23630/1"/>
-<part name="R1" library="rcl" library_urn="urn:adsk.eagle:library:334" deviceset="R-US_" device="0204/2V" package3d_urn="urn:adsk.eagle:package:23495/1"/>
-<part name="R2" library="rcl" library_urn="urn:adsk.eagle:library:334" deviceset="R-US_" device="0204/2V" package3d_urn="urn:adsk.eagle:package:23495/1"/>
+<part name="C3" library="rcl" library_urn="urn:adsk.eagle:library:334" deviceset="C-EU" device="025-024X044" package3d_urn="urn:adsk.eagle:package:23630/1" value="100u"/>
+<part name="R1" library="rcl" library_urn="urn:adsk.eagle:library:334" deviceset="R-US_" device="0204/2V" package3d_urn="urn:adsk.eagle:package:23495/1" value="904"/>
+<part name="R2" library="rcl" library_urn="urn:adsk.eagle:library:334" deviceset="R-US_" device="0204/2V" package3d_urn="urn:adsk.eagle:package:23495/1" value="285"/>
 <part name="X_4" library="ngspice-simulation" library_urn="urn:adsk.eagle:library:527439" deviceset="GND" device=""/>
-<part name="T1" library="transistor" library_urn="urn:adsk.eagle:library:402" deviceset="2N3440" device="" package3d_urn="urn:adsk.eagle:package:28729/1" value=""/>
-<part name="R3" library="rcl" library_urn="urn:adsk.eagle:library:334" deviceset="R-US_" device="0204/2V" package3d_urn="urn:adsk.eagle:package:23495/1"/>
-<part name="R4" library="rcl" library_urn="urn:adsk.eagle:library:334" deviceset="R-US_" device="0204/2V" package3d_urn="urn:adsk.eagle:package:23495/1"/>
+<part name="T1" library="transistor" library_urn="urn:adsk.eagle:library:402" deviceset="2N3440" device="" package3d_urn="urn:adsk.eagle:package:28729/1" value="SC 945"/>
+<part name="R3" library="rcl" library_urn="urn:adsk.eagle:library:334" deviceset="R-US_" device="0204/2V" package3d_urn="urn:adsk.eagle:package:23495/1" value="25"/>
+<part name="R4" library="rcl" library_urn="urn:adsk.eagle:library:334" deviceset="R-US_" device="0204/2V" package3d_urn="urn:adsk.eagle:package:23495/1" value="125"/>
 <part name="P+2" library="supply1" library_urn="urn:adsk.eagle:library:371" deviceset="+5V" device=""/>
 <part name="D1" library="diode" library_urn="urn:adsk.eagle:library:210" deviceset="1N4004" device="" package3d_urn="urn:adsk.eagle:package:43336/1"/>
@@
 <part name="P+3" library="supply1" library_urn="urn:adsk.eagle:library:371" deviceset="+5V" device=""/>
 <part name="X_6" library="ngspice-simulation" library_urn="urn:adsk.eagle:library:527439" deviceset="GND" device=""/>
-<part name="OK1" library="optocoupler" library_urn="urn:adsk.eagle:library:320" deviceset="SFH618?*" device="A" package3d_urn="urn:adsk.eagle:package:21960/1" technology="-2"/>
-<part name="R8" library="rcl" library_urn="urn:adsk.eagle:library:334" deviceset="R-US_" device="0204/2V" package3d_urn="urn:adsk.eagle:package:23495/1"/>
+<part name="OK1" library="optocoupler" library_urn="urn:adsk.eagle:library:320" deviceset="SFH618?*" device="A" package3d_urn="urn:adsk.eagle:package:21960/1" technology="-2" value="LTV817"/>
+<part name="R8" library="rcl" library_urn="urn:adsk.eagle:library:334" deviceset="R-US_" device="0204/2V" package3d_urn="urn:adsk.eagle:package:23495/1" value="220"/>
 <part name="P+4" library="supply1" library_urn="urn:adsk.eagle:library:371" deviceset="VCC" device="" value="+13.8V"/>
 <part name="X1" library="con-avx" library_urn="urn:adsk.eagle:library:129" deviceset="00917?002" device="6" package3d_urn="urn:adsk.eagle:package:6130/1" value="PTT"/>
@@
 <part name="X_8" library="ngspice-simulation" library_urn="urn:adsk.eagle:library:527439" deviceset="GND" device=""/>
 <part name="LED1" library="led" library_urn="urn:adsk.eagle:library:259" deviceset="*P4" device="-TOP" package3d_urn="urn:adsk.eagle:package:15879/1" technology="LA" value=""/>
-<part name="R10" library="rcl" library_urn="urn:adsk.eagle:library:334" deviceset="R-US_" device="0204/2V" package3d_urn="urn:adsk.eagle:package:23495/1"/>
+<part name="R10" library="rcl" library_urn="urn:adsk.eagle:library:334" deviceset="R-US_" device="0204/2V" package3d_urn="urn:adsk.eagle:package:23495/1" value="150"/>
 </parts>
 <sheets>
@@
 <text x="-60.96" y="68.58" size="1.778" layer="91" grouprefs="PC_TO_RADIO">right (VOX)</text>
 <text x="-60.96" y="66.04" size="1.778" layer="91" grouprefs="PC_TO_RADIO">left (Audio)</text>
+<text x="5.08" y="78.74" size="1.778" layer="91">Ic = 20mA</text>
 </plain>
 <instances>
@@
 <instance part="T1" gate="G$1" x="-2.54" y="68.58" smashed="yes" grouprefs="VOX">
 <attribute name="NAME" x="-12.7" y="76.2" size="1.778" layer="95"/>
-<attribute name="VALUE" x="-12.7" y="73.66" size="1.778" layer="96"/>
+<attribute name="VALUE" x="0" y="68.58" size="1.778" layer="96"/>
 </instance>
 <instance part="R3" gate="G$1" x="0" y="58.42" smashed="yes" rot="R90" grouprefs="VOX">
@@
 <wire x1="55.88" y1="48.26" x2="58.42" y2="48.26" width="0.1524" layer="91"/>
 <wire x1="129.54" y1="50.8" x2="129.54" y2="30.48" width="0.1524" layer="91"/>
-<wire x1="129.54" y1="30.48" x2="55.88" y2="30.48" width="0.1524" layer="91"/>
+<wire x1="129.54" y1="30.48" x2="101.6" y2="30.48" width="0.1524" layer="91"/>
+<wire x1="101.6" y1="30.48" x2="55.88" y2="30.48" width="0.1524" layer="91"/>
 <wire x1="55.88" y1="30.48" x2="55.88" y2="48.26" width="0.1524" layer="91"/>
 <junction x="55.88" y="48.26"/>
+<pinref part="U$1" gate="G$1" pin="GND2"/>
+<wire x1="91.44" y1="53.34" x2="101.6" y2="53.34" width="0.1524" layer="91"/>
+<wire x1="101.6" y1="53.34" x2="101.6" y2="30.48" width="0.1524" layer="91"/>
+<junction x="101.6" y="30.48"/>
 </segment>
 <segment>

Commit message: Transistor Amp Caluclations | Schottky diode
Parts:
- C4: value (none) -> 100u
- D1: value 1N4004 -> 1N4007
- R1: value 904 -> 1k
- R2: value 285 -> 220
- R3: value 25 -> 10
- R4: value 125 -> 100
- R5: value (none) -> 2k
- T1: value SC 945 -> PN2222A
Changed lines of the file:
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@@
 <part name="P+1" library="supply1" library_urn="urn:adsk.eagle:library:371" deviceset="+5V" device=""/>
 <part name="C3" library="rcl" library_urn="urn:adsk.eagle:library:334" deviceset="C-EU" device="025-024X044" package3d_urn="urn:adsk.eagle:package:23630/1" value="100u"/>
-<part name="R1" library="rcl" library_urn="urn:adsk.eagle:library:334" deviceset="R-US_" device="0204/2V" package3d_urn="urn:adsk.eagle:package:23495/1" value="904"/>
-<part name="R2" library="rcl" library_urn="urn:adsk.eagle:library:334" deviceset="R-US_" device="0204/2V" package3d_urn="urn:adsk.eagle:package:23495/1" value="285"/>
+<part name="R1" library="rcl" library_urn="urn:adsk.eagle:library:334" deviceset="R-US_" device="0204/2V" package3d_urn="urn:adsk.eagle:package:23495/1" value="1k"/>
+<part name="R2" library="rcl" library_urn="urn:adsk.eagle:library:334" deviceset="R-US_" device="0204/2V" package3d_urn="urn:adsk.eagle:package:23495/1" value="220"/>
 <part name="X_4" library="ngspice-simulation" library_urn="urn:adsk.eagle:library:527439" deviceset="GND" device=""/>
-<part name="T1" library="transistor" library_urn="urn:adsk.eagle:library:402" deviceset="2N3440" device="" package3d_urn="urn:adsk.eagle:package:28729/1" value="SC 945"/>
-<part name="R3" library="rcl" library_urn="urn:adsk.eagle:library:334" deviceset="R-US_" device="0204/2V" package3d_urn="urn:adsk.eagle:package:23495/1" value="25"/>
-<part name="R4" library="rcl" library_urn="urn:adsk.eagle:library:334" deviceset="R-US_" device="0204/2V" package3d_urn="urn:adsk.eagle:package:23495/1" value="125"/>
+<part name="T1" library="transistor" library_urn="urn:adsk.eagle:library:402" deviceset="2N3440" device="" package3d_urn="urn:adsk.eagle:package:28729/1" value="PN2222A"/>
+<part name="R3" library="rcl" library_urn="urn:adsk.eagle:library:334" deviceset="R-US_" device="0204/2V" package3d_urn="urn:adsk.eagle:package:23495/1" value="10"/>
+<part name="R4" library="rcl" library_urn="urn:adsk.eagle:library:334" deviceset="R-US_" device="0204/2V" package3d_urn="urn:adsk.eagle:package:23495/1" value="100"/>
 <part name="P+2" library="supply1" library_urn="urn:adsk.eagle:library:371" deviceset="+5V" device=""/>
-<part name="D1" library="diode" library_urn="urn:adsk.eagle:library:210" deviceset="1N4004" device="" package3d_urn="urn:adsk.eagle:package:43336/1"/>
-<part name="C4" library="rcl" library_urn="urn:adsk.eagle:library:334" deviceset="C-EU" device="025-024X044" package3d_urn="urn:adsk.eagle:package:23630/1"/>
+<part name="D1" library="diode" library_urn="urn:adsk.eagle:library:210" deviceset="1N4004" device="" package3d_urn="urn:adsk.eagle:package:43336/1" value="1N4007"/>
+<part name="C4" library="rcl" library_urn="urn:adsk.eagle:library:334" deviceset="C-EU" device="025-024X044" package3d_urn="urn:adsk.eagle:package:23630/1" value="100u"/>
 <part name="X_5" library="ngspice-simulation" library_urn="urn:adsk.eagle:library:527439" deviceset="GND" device=""/>
-<part name="R5" library="rcl" library_urn="urn:adsk.eagle:library:334" deviceset="R-US_" device="0204/2V" package3d_urn="urn:adsk.eagle:package:23495/1"/>
+<part name="R5" library="rcl" library_urn="urn:adsk.eagle:library:334" deviceset="R-US_" device="0204/2V" package3d_urn="urn:adsk.eagle:package:23495/1" value="2k"/>
 <part name="R6" library="rcl" library_urn="urn:adsk.eagle:library:334" deviceset="POTENTIOMETER_" device="PT-10S" package3d_urn="urn:adsk.eagle:package:23785/1"/>
 <part name="R7" library="rcl" library_urn="urn:adsk.eagle:library:334" deviceset="POTENTIOMETER_" device="PT-10S" package3d_urn="urn:adsk.eagle:package:23785/1"/>
@@
 <instance part="R1" gate="G$1" x="-10.16" y="73.66" smashed="yes" rot="R90" grouprefs="VOX">
 <attribute name="NAME" x="-11.6586" y="69.85" size="1.778" layer="95" rot="R90"/>
-<attribute name="VALUE" x="-6.858" y="69.85" size="1.778" layer="96" rot="R90"/>
+<attribute name="VALUE" x="-6.35" y="74.422" size="1.778" layer="96" rot="R180"/>
 </instance>
 <instance part="R2" gate="G$1" x="-10.16" y="63.5" smashed="yes" rot="R90" grouprefs="VOX">
 <attribute name="NAME" x="-11.6586" y="59.69" size="1.778" layer="95" rot="R90"/>
-<attribute name="VALUE" x="-6.858" y="59.69" size="1.778" layer="96" rot="R90"/>
+<attribute name="VALUE" x="-3.81" y="64.262" size="1.778" layer="96" rot="R180"/>
 </instance>
 <instance part="X_4" gate="G$1" x="-10.16" y="48.26" smashed="yes" grouprefs="VOX"/>
@@
 <instance part="R3" gate="G$1" x="0" y="58.42" smashed="yes" rot="R90" grouprefs="VOX">
 <attribute name="NAME" x="-1.4986" y="54.61" size="1.778" layer="95" rot="R90"/>
-<attribute name="VALUE" x="3.302" y="54.61" size="1.778" layer="96" rot="R90"/>
+<attribute name="VALUE" x="3.81" y="56.642" size="1.778" layer="96" rot="R180"/>
 </instance>
 <instance part="R4" gate="G$1" x="0" y="78.74" smashed="yes" rot="R90" grouprefs="VOX">
 <attribute name="NAME" x="-1.4986" y="74.93" size="1.778" layer="95" rot="R90"/>
-<attribute name="VALUE" x="3.302" y="74.93" size="1.778" layer="96" rot="R90"/>
+<attribute name="VALUE" x="-1.27" y="82.042" size="1.778" layer="96" rot="R180"/>
 </instance>
 <instance part="P+2" gate="1" x="0" y="91.44" smashed="yes" grouprefs="VOX">
@@
 <instance part="C4" gate="G$1" x="22.86" y="68.58" smashed="yes" rot="R180" grouprefs="VOX">
 <attribute name="NAME" x="21.336" y="68.199" size="1.778" layer="95" rot="R180"/>
-<attribute name="VALUE" x="21.336" y="73.279" size="1.778" layer="96" rot="R180"/>
+<attribute name="VALUE" x="21.336" y="65.659" size="1.778" layer="96" rot="R180"/>
 </instance>
 <instance part="X_5" gate="G$1" x="22.86" y="60.96" smashed="yes" grouprefs="VOX"/>
 <instance part="R5" gate="G$1" x="30.48" y="68.58" smashed="yes" rot="R90" grouprefs="VOX">
 <attribute name="NAME" x="28.9814" y="64.77" size="1.778" layer="95" rot="R90"/>
-<attribute name="VALUE" x="33.782" y="64.77" size="1.778" layer="96" rot="R90"/>
+<attribute name="VALUE" x="34.29" y="66.802" size="1.778" layer="96" rot="R180"/>
 </instance>
 <instance part="R6" gate="1" x="40.64" y="2.54" smashed="yes" rot="R90" grouprefs="CONTROLL_POTENTIOMETERS">
